File: PicoCalcPiZeroKiCAD/PicoCalcPiZero.kicad_pcb (KiCad board)
At the start: 2 copper layers, 33.5 x 52.5 mm, 2 parts, among them J2 Raspberry_Pi_2_3

Commit message: Add files via upload
Parts:
- moved J2 13.0 mm to (94.5, 78.9)
Routing:
- net SPI1_CS: track 34.5 -> 6.62 mm
- net LCD_DC: track 28.3 -> 15.5 mm
- net LCD_RST: track 25.7 -> 14.5 mm
- net I2C1_SCL: track 22.9 -> 12.0 mm
- net I2C1_SDA: track 22.7 -> 11.8 mm
- net PWM_L: track 32.6 -> 42.6 mm
- net PWM_R: track 35.1 -> 44.9 mm
- net SPI1_TX: track 21.0 -> 12.8 mm
- net GND: track 26.5 -> 29.7 mm
- net VSYS: track 26.0 -> 28.6 mm
Other:
- board size 33.5 x 52.5 mm -> 32 x 65.5 mm
- board text added: "Header and SBC on other Side!"
- board text removed: "Header and SBC on the other side!"
